Commit message: Both back and front legs complete

File: body.urdf (robot description, URDF)
Before this commit: robot robot, 3 links, 2 joints
Links:
- added link Back_Lower_Leg, mass 1; collision box size=0.2 0.2 1.0; visual box size=0.2 0.2 1.0
- added link Front_Lower_Leg, mass 1; collision box size=0.2 0.2 1.0; visual box size=0.2 0.2 1.0
- added link Left_Leg, mass 1; collision box size=1.0 0.2 0.2; visual box size=1.0 0.2 0.2
- added link Right_Leg, mass 1; collision box size=1.0 0.2 0.2; visual box size=1.0 0.2 0.2
- link Back_Leg: geometry collision box size=0.2 1.0 0.2; visual box size=0.2 1.0 0.2
- link Front_Leg: geometry collision box size=0.2 1.0 0.2; visual box size=0.2 1.0 0.2
Joints:
- added joint Back_Leg_Lower_Leg: type revolute, parent Back_Leg, child Back_Lower_Leg, origin xyz=0.0, -1.0, 0.0 rpy=0 0 0, axis 1 0 0, limit lower=-3.14159 upper=3.14159 effort=0.0 velocity=0.0
- added joint Front_Leg_Lower_Leg: type revolute, parent Front_Leg, child Front_Lower_Leg, origin xyz=0.0, 1.0, 0.0 rpy=0 0 0, axis 1 0 0, limit lower=-3.14159 upper=3.14159 effort=0.0 velocity=0.0
- added joint Torso_Left_Leg: type revolute, parent Torso, child Left_Leg, origin xyz=-0.5, 0.0, 1.0 rpy=0 0 0, axis 0 1 0, limit lower=-3.14159 upper=3.14159 effort=0.0 velocity=0.0
- added joint Torso_Right_Leg: type revolute, parent Torso, child Right_Leg, origin xyz=0.5, 0.0, 1.0 rpy=0 0 0, axis 0 1 0, limit lower=-3.14159 upper=3.14159 effort=0.0 velocity=0.0
- joint Torso_Back_Leg: axis 0 1 0 -> 1 0 0; origin xyz=1.0, 0.0, 1.0 rpy=0 0 0 -> xyz=0.0, -0.5, 1.0 rpy=0 0 0
- joint Torso_Front_Leg: axis 0 1 0 -> 1 0 0; origin xyz=2.0, 0.0, 1.0 rpy=0 0 0 -> xyz=0, 0.5, 1.0 rpy=0 0 0

Commit message: Quadraped (robot) complete

File: body.urdf (robot description, URDF)
Before this commit: robot robot, 7 links, 6 joints
Links:
- added link Left_Lower_Leg, mass 1; collision box size=0.2 0.2 1.0; visual box size=0.2 0.2 1.0
- added link Right_Lower_Leg, mass 1; collision box size=0.2 0.2 1.0; visual box size=0.2 0.2 1.0
Joints:
- added joint Left_Leg_Lower_Leg: type revolute, parent Left_Leg, child Left_Lower_Leg, origin xyz=-1.0, 0 0.0, 0.0 rpy=0 0 0, axis 0 1 0, limit lower=-3.14159 upper=3.14159 effort=0.0 velocity=0.0
- added joint Right_Leg_Lower_Leg: type revolute, parent Right_Leg, child Right_Lower_Leg, origin xyz=1.0, 0.0, 0.0 rpy=0 0 0, axis 0 1 0, limit lower=-3.14159 upper=3.14159 effort=0.0 velocity=0.0

Commit message: Want to encourage oscilliatory behavior

File: body.urdf (robot description, URDF)
Before this commit: robot robot, 9 links, 8 joints
Links:
- link Back_Lower_Leg: geometry collision box size=0.2 0.2 0.28883744571674963; visual box size=0.2 0.2 0.28883744571674963
- link Front_Lower_Leg: geometry collision box size=0.2 0.2 0.28883744571674963; visual box size=0.2 0.2 0.28883744571674963
- link Left_Lower_Leg: geometry collision box size=0.2 0.2 0.28883744571674963; visual box size=0.2 0.2 0.28883744571674963
- link Right_Lower_Leg: geometry collision box size=0.2 0.2 0.28883744571674963; visual box size=0.2 0.2 0.28883744571674963
Joints:
- joint Torso_Back_Leg: origin xyz=0.0, -0.5, 1.0 rpy=0 0 0 -> xyz=0.0, -0.5, 0.28883744571674963 rpy=0 0 0
- joint Torso_Front_Leg: origin xyz=0, 0.5, 1.0 rpy=0 0 0 -> xyz=0, 0.5, 0.28883744571674963 rpy=0 0 0
- joint Torso_Left_Leg: origin xyz=-0.5, 0.0, 1.0 rpy=0 0 0 -> xyz=-0.5, 0.0, 0.28883744571674963 rpy=0 0 0
- joint Torso_Right_Leg: origin xyz=0.5, 0.0, 1.0 rpy=0 0 0 -> xyz=0.5, 0.0, 0.28883744571674963 rpy=0 0 0

Commit message: Long legs

File: body.urdf (robot description, URDF)
Before this commit: robot robot, 9 links, 8 joints
Links:
- link Back_Lower_Leg: geometry collision box size=0.2 0.2 2.6796953107058914; visual box size=0.2 0.2 2.6796953107058914
- link Front_Lower_Leg: geometry collision box size=0.2 0.2 2.6796953107058914; visual box size=0.2 0.2 2.6796953107058914
- link Left_Lower_Leg: geometry collision box size=0.2 0.2 2.6796953107058914; visual box size=0.2 0.2 2.6796953107058914
- link Right_Lower_Leg: geometry collision box size=0.2 0.2 2.6796953107058914; visual box size=0.2 0.2 2.6796953107058914
Joints:
- joint Torso_Back_Leg: origin xyz=0.0, -0.5, 0.28883744571674963 rpy=0 0 0 -> xyz=0.0, -0.5, 2.6796953107058914 rpy=0 0 0
- joint Torso_Front_Leg: origin xyz=0, 0.5, 0.28883744571674963 rpy=0 0 0 -> xyz=0, 0.5, 2.6796953107058914 rpy=0 0 0
- joint Torso_Left_Leg: origin xyz=-0.5, 0.0, 0.28883744571674963 rpy=0 0 0 -> xyz=-0.5, 0.0, 2.6796953107058914 rpy=0 0 0
- joint Torso_Right_Leg: origin xyz=0.5, 0.0, 0.28883744571674963 rpy=0 0 0 -> xyz=0.5, 0.0, 2.6796953107058914 rpy=0 0 0

Commit message: Alpha test, writing to fitness file

File: body.urdf (robot description, URDF)
Before this commit: robot robot, 3 links, 2 joints
Joints:
- joint Torso_Back_Leg: axis 0 1 0 -> 0.0, 1.0, 0.0
- joint Torso_Front_Leg: axis 0 1 0 -> 0.0, 1.0, 0.0
